File: WifiTick.sch (KiCad schematic (older format))
At the start: 30 parts, among them P1 CONN_01X01, U1 TPS73533, U2 ESP8266, U3 25Q32, X1 26MHz

Commit message: Update due to new KiCad version.
Parts:
- A1: symbol ANT -> WifiTickLibrary:ANT
- C1, C2, C3, C4, C5, C6, C7, C8: symbol C -> WifiTick-rescue:C
- D1: symbol LED_ALT -> WifiTick-rescue:LED_ALT
- H1: symbol header20 -> WifiTickLibrary:header20
- P1: symbol CONN_01X01 -> WifiTick-rescue:CONN_01X01
- R1, R10, R11, R12, R13, R14, R2, R3, R4, R5, R6, R7, R8, R9: symbol R -> WifiTick-rescue:R
- U1: symbol TPS735 -> WifiTickLibrary:TPS735
- U2: symbol ESP8266 -> WifiTickLibrary:ESP8266
- U3: symbol 25Q32 -> WifiTickLibrary:25Q32
- X1: symbol CRYSTAL_SMD -> WifiTick-rescue:CRYSTAL_SMD
Connections:
- wire segments 83 -> 104
Other:
- moved on the sheet: C1, C3
